File: 4_relay_5Switch.brd (EAGLE design)
At the start: 54 x 78.7 mm, 13 parts, among them U1 NCP1117ST50T3G

Commit message: working on
Parts:
- added LED1, LED2: (no value), adafruit:CHIP-LED0805
- added R1, R2: (no value), resistor:R0805
- C2: value 100n -> 1.0uF; device SmartPrj:C0603-ROUND -> SparkFun-Capacitors:0805
- moved S2 5.39 mm to (34.5, 69.8)
- moved S5 5.07 mm to (33.3, 11.6)
- moved S1 4.58 mm to (34.5, 52.1)
- moved S3 4.58 mm to (34.5, 31.8)
- moved S4 2.54 mm to (5.33, 71.1)
Connections:
- new net N$11: R2.1, U$2.3
- new net N$12: R1.1, U$2.2
- new net N$13: LED1.A, R2.2
- new net N$14: LED2.A, R1.2
- net +5V: no longer U1.4
- net GND: now also LED1.C, LED2.C
Routing:
- net GND: track 193.0 -> 93.5 mm, vias 1 -> 2
- net N$12: track 0.00 -> 23.8 mm
- net N$11: track 0.00 -> 19.2 mm
- net VIN: track 151.0 -> 141.1 mm
- net N$3: track 64.5 -> 55.0 mm
- net N$1: track 50.8 -> 44.8 mm
- net N$5: track 37.3 -> 32.1 mm
- net N$13: track 0.00 -> 2.90 mm
- net N$9: track 35.3 -> 32.5 mm
- net N$14: track 0.00 -> 2.58 mm
- net +5V: track 36.7 -> 39.0 mm
- net N$10: track 46.7 -> 46.0 mm
- removed copper zone on layer 1, net +5V
- removed copper zone on layer 1, net TEST
Other:
- board size 54 x 78.7 mm -> 50.8 x 76.2 mm
