File: 4_relay_5Switch.sch (EAGLE design)
At the start: 13 parts, among them U1 NCP1117ST50T3G

Commit message: working on
Parts:
- added LED1, LED2: (no value), adafruit:LEDCHIP-LED0805
- added R1, R2: (no value), resistor:R-US_R0805
- C2: value 100n -> 1.0uF; device SmartPrj:C-EU0603-RND -> SparkFun-Capacitors:1.0UF-25V-+80/-20(0805)
Connections:
- new net N$11: R2.1, U$2.(PCINT9/XTAL2)PB1
- new net N$12: R1.1, U$2.(PCINT8/XTAL1/CLKI)PB0
- new net N$13: LED1.A, R2.2
- new net N$14: LED2.A, R1.2
- net +5V: no longer U1.OUT
- net GND: now also LED1.C, LED2.C
Other:
- moved on the sheet: C2
Changed lines of the file:
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@@
 <part name="U$2" library="SparkFun-DigitalIC" deviceset="ATTINY84" device=""/>
 <part name="S3" library="SparkFun-Electromechanical_alr" deviceset="SWITCH-MOMENTARY-2" device=""/>
-<part name="C2" library="SmartPrj" deviceset="C-EU" device="0603-RND" value="100n"/>
+<part name="C2" library="SparkFun-Capacitors" deviceset="1.0UF-25V-+80/-20(0805)" device="" value="1.0uF"/>
 <part name="GND7" library="supply1" deviceset="GND" device=""/>
 <part name="PC1" library="rcl" deviceset="CPOL-EU" device="E2.5-5V" value="47u"/>
@@
 <part name="JP1" library="SparkFun-Connectors" deviceset="M06" device="NO_SILK_FEMALE_PTH"/>
 <part name="PC2" library="rcl" deviceset="CPOL-EU" device="E2.5-5V" value="47u"/>
+<part name="LED1" library="adafruit" deviceset="LED" device="CHIP-LED0805"/>
+<part name="LED2" library="adafruit" deviceset="LED" device="CHIP-LED0805"/>
+<part name="GND1" library="supply1" deviceset="GND" device=""/>
+<part name="R1" library="resistor" deviceset="R-US_" device="R0805"/>
+<part name="R2" library="resistor" deviceset="R-US_" device="R0805"/>
 </parts>
 <sheets>
@@
 <attribute name="VALUE" x="119.38" y="15.24" size="1.778" layer="96"/>
 </instance>
+<instance part="LED1" gate="G$1" x="116.84" y="116.84" rot="R90"/>
+<instance part="LED2" gate="G$1" x="116.84" y="109.22" rot="R90"/>
+<instance part="GND1" gate="1" x="137.16" y="111.76"/>
+<instance part="R1" gate="G$1" x="106.68" y="114.3"/>
+<instance part="R2" gate="G$1" x="106.68" y="116.84"/>
 </instances>
 <busses>
@@
 <wire x1="99.06" y1="22.86" x2="106.68" y2="22.86" width="0.1524" layer="91"/>
 <wire x1="88.9" y1="25.4" x2="99.06" y2="25.4" width="0.1524" layer="91"/>
-<wire x1="88.9" y1="27.94" x2="99.06" y2="27.94" width="0.1524" layer="91"/>
-<wire x1="99.06" y1="27.94" x2="99.06" y2="25.4" width="0.1524" layer="91"/>
 <wire x1="99.06" y1="25.4" x2="99.06" y2="22.86" width="0.1524" layer="91"/>
 <wire x1="106.68" y1="22.86" x2="114.3" y2="22.86" width="0.1524" layer="91"/>
-<wire x1="114.3" y1="22.86" x2="114.3" y2="20.32" width="0.1524" layer="91"/>
-<junction x="99.06" y="25.4"/>
+<wire x1="114.3" y1="22.86" x2="114.3" y2="17.78" width="0.1524" layer="91"/>
 <junction x="106.68" y="22.86"/>
 <pinref part="P+8" gate="1" pin="+5V"/>
 <pinref part="U1" gate="G$1" pin="OUT@1"/>
-<pinref part="U1" gate="G$1" pin="OUT"/>
 <pinref part="C2" gate="G$1" pin="2"/>
 <pinref part="PC2" gate="G$1" pin="+"/>
@@
 </segment>
 <segment>
-<wire x1="114.3" y1="12.7" x2="114.3" y2="10.16" width="0.1524" layer="91"/>
 <pinref part="C2" gate="G$1" pin="1"/>
 <pinref part="GND7" gate="1" pin="GND"/>
 <pinref part="PC2" gate="G$1" pin="-"/>
-<wire x1="127" y1="12.7" x2="114.3" y2="12.7" width="0.1524" layer="91"/>
-<junction x="114.3" y="12.7"/>
+<wire x1="127" y1="12.7" x2="114.3" y2="10.16" width="0.1524" layer="91"/>
+<junction x="114.3" y="10.16"/>
 </segment>
 <segment>
@@
 <pinref part="GND9" gate="1" pin="GND"/>
 <pinref part="PC1" gate="G$1" pin="-"/>
+</segment>
+<segment>
+<pinref part="GND1" gate="1" pin="GND"/>
+<wire x1="137.16" y1="114.3" x2="137.16" y2="116.84" width="0.1524" layer="91"/>
+<pinref part="LED2" gate="G$1" pin="C"/>
+<wire x1="121.92" y1="109.22" x2="127" y2="109.22" width="0.1524" layer="91"/>
+<wire x1="127" y1="109.22" x2="127" y2="114.3" width="0.1524" layer="91"/>
+<pinref part="LED1" gate="G$1" pin="C"/>
+<wire x1="127" y1="116.84" x2="127" y2="119.38" width="0.1524" layer="91"/>
+<wire x1="127" y1="119.38" x2="121.92" y2="119.38" width="0.1524" layer="91"/>
+<wire x1="121.92" y1="119.38" x2="121.92" y2="116.84" width="0.1524" layer="91"/>
+<wire x1="137.16" y1="116.84" x2="127" y2="116.84" width="0.1524" layer="91"/>
+<wire x1="127" y1="116.84" x2="127" y2="114.3" width="0.1524" layer="91"/>
 </segment>
 </net>
@@
 </segment>
 </net>
+<net name="N$11" class="0">
+<segment>
+<pinref part="U$2" gate="G$1" pin="(PCINT9/XTAL2)PB1"/>
+<wire x1="76.2" y1="116.84" x2="101.6" y2="116.84" width="0.1524" layer="91"/>
+<pinref part="R2" gate="G$1" pin="1"/>
+</segment>
+</net>
+<net name="N$12" class="0">
+<segment>
+<pinref part="U$2" gate="G$1" pin="(PCINT8/XTAL1/CLKI)PB0"/>
+<wire x1="76.2" y1="114.3" x2="101.6" y2="114.3" width="0.1524" layer="91"/>
+<pinref part="R1" gate="G$1" pin="1"/>
+</segment>
+</net>
+<net name="N$14" class="0">
+<segment>
+<pinref part="LED2" gate="G$1" pin="A"/>
+<pinref part="R1" gate="G$1" pin="2"/>
+<wire x1="111.76" y1="114.3" x2="114.3" y2="114.3" width="0.1524" layer="91"/>
+<wire x1="114.3" y1="114.3" x2="114.3" y2="109.22" width="0.1524" layer="91"/>
+</segment>
+</net>
+<net name="N$13" class="0">
+<segment>
+<pinref part="LED1" gate="G$1" pin="A"/>
+<pinref part="R2" gate="G$1" pin="2"/>
+<wire x1="111.76" y1="116.84" x2="114.3" y2="116.84" width="0.1524" layer="91"/>
+</segment>
+</net>
